File: Electrónica/Helios/Helios_PCB/Helios_PCB/Helios_PCB.kicad_pcb (KiCad board)
At the start: 2 copper layers, 15 x 30.3 mm, 11 parts, among them J0 Conn_01x05_Male, Q0 AO3400A, U0 OPA2380

Commit message: Helios: Second Iter
Parts:
- moved J0 57.5 mm to (153.8, 95.5)
- moved Q0 57.5 mm to (144.3, 99.5)
- moved R2 57.5 mm to (144.3, 93.9)
- moved R3 57.5 mm to (144.3, 96.9)
- moved D0 57.5 mm to (147.8, 89.8)
- moved D1 57.5 mm to (147.8, 109.2)
- moved F0 57.5 mm to (147.8, 89.8)
- moved F1 57.5 mm to (147.8, 109.2)
- moved R0 57.5 mm to (145.3, 93.5)
- moved R1 57.5 mm to (145.3, 105.5)
- moved U0 57.5 mm to (143.8, 99.5)
Routing:
- net GND: vias 2 -> 1
