File: Electrónica/Helios/Helios_PCB/Helios_PCB/Helios_PCB.kicad_sch (KiCad schematic)
At the start: 11 parts, among them J0 Conn_01x05_Male, Q0 AO3400A, U0 OPA2380

Commit message: Helios: Second Iter
Parts:
- removed J0: Conn_01x05_Male, Connector_PinHeader_2.00mm:PinHeader_1x05_P2.00mm_Vertical, symbol Connector:Conn_01x05_Male
- added D2, D3: LED, LED_SMD:LED_PLCC-2, symbol Device:LED
- added F2, F3: SFH2704, Helios:SFH2704_Photodiode, symbol Helios:SFH2704
- added R2, R3: Rf, Helios:RS_0805, symbol Device:R
- added U1: OPA2380, Helios:OPA2380, symbol Helios:OPA2380
Connections:
- net GND: now also F2.2 (A), F3.2 (A), U1.3 (+IA), U1.4 (GND), U1.5 (+IB)
- net VCC: now also U1.8 (VCC)
- net at D1.1 (K): now also D2.2 (A); no longer Q0.3 (D)
- new net: D2.1 (K), D3.2 (A)
- new net: F2.1 (K), R2.2, U1.2 (-IA)
- new net: F3.1 (K), R3.2, U1.6 (-IB)
- new net: D3.1 (K), Q0.3 (D)
- new net O2: R2.1, U1.1 (OA)
- new net O3: R3.1, U1.7 (OB)
Other:
- moved on the sheet: Q0, R3
