File: Electrónica/Helios/Helios_PCB/Helios_PCB_emitter/Helios_PCB.kicad_pcb (KiCad board)
At the start: 2 copper layers, 15 x 30.3 mm, 11 parts, among them J0 Conn_01x05_Male, Q0 AO3400A, U0 OPA2380

Commit message: Helios: Iteration3
Parts:
- added D2: LED, LED_SMD:LED_PLCC-2, F.Cu at (188.3, 94.9)
- added D3: LED, LED_SMD:LED_PLCC-2, F.Cu at (188.3, 99.7)
- added F2: SFH2704, Helios:SFH2704_Photodiode, F.Cu at (192.8, 98.5)
- added F3: SFH2704, Helios:SFH2704_Photodiode, F.Cu at (196.4, 93.9)
- added R2: Rf, Helios:RS_0805, F.Cu at (193.1, 93.7)
- added R3: Rf, Helios:RS_0805, F.Cu at (193.1, 96.0)
- added U1: OPA2380, Helios:OPA2380, F.Cu at (183.4, 96.0)
- renumbered R2 to R4, R3 to R5
Connections:
- Q0 pad 3: Net-(D1-Pad1) -> Net-(D3-Pad1)
Routing:
- net Net-(D3-Pad1): track 0.00 -> 10.9 mm
- net Net-(D1-Pad1): track 10.9 -> 0.00 mm
