File: Electrónica/Helios/Helios_PCB/Helios_PCB_emitter/Helios_PCB.kicad_sch (KiCad schematic)
At the start: 17 parts, among them Q0 AO3400A, U0 OPA2380, U1 OPA2380

Commit message: Helios: Iteration3
Parts:
- renumbered R2 to R4, R3 to R5
Changed lines of the file:
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@@
   (symbol (lib_id "power:GND") (at 38.1 140.97 0) (unit 1)
     (in_bom yes) (on_board yes)
-    (property "Reference" "#PWR?" (id 0) (at 38.1 147.32 0)
+    (property "Reference" "#PWR0104" (id 0) (at 38.1 147.32 0)
       (effects (font (size 1.27 1.27)) hide)
     )
@@
   (symbol (lib_id "Device:R") (at 153.67 99.06 0) (unit 1)
     (in_bom yes) (on_board yes) (fields_autoplaced)
-    (property "Reference" "R3" (id 0) (at 155.448 99.4938 0)
+    (property "Reference" "R5" (id 0) (at 155.448 99.4938 0)
       (effects (font (size 1.27 1.27)) (justify left))
     )
@@
   (symbol (lib_id "power:VCC") (at 76.2 106.68 0) (unit 1)
     (in_bom yes) (on_board yes)
-    (property "Reference" "#PWR?" (id 0) (at 76.2 110.49 0)
+    (property "Reference" "#PWR0102" (id 0) (at 76.2 110.49 0)
       (effects (font (size 1.27 1.27)) hide)
     )
@@
   (symbol (lib_id "Device:R") (at 168.91 41.91 180) (unit 1)
     (in_bom yes) (on_board yes) (fields_autoplaced)
-    (property "Reference" "R2" (id 0) (at 170.688 42.3438 0)
+    (property "Reference" "R4" (id 0) (at 170.688 42.3438 0)
       (effects (font (size 1.27 1.27)) (justify right))
     )
@@
   (symbol (lib_id "power:GND") (at 88.9 140.97 0) (unit 1)
     (in_bom yes) (on_board yes)
-    (property "Reference" "#PWR?" (id 0) (at 88.9 147.32 0)
+    (property "Reference" "#PWR0101" (id 0) (at 88.9 147.32 0)
       (effects (font (size 1.27 1.27)) hide)
     )
@@
   (symbol (lib_id "power:GND") (at 76.2 121.92 0) (unit 1)
     (in_bom yes) (on_board yes)
-    (property "Reference" "#PWR?" (id 0) (at 76.2 128.27 0)
+    (property "Reference" "#PWR0103" (id 0) (at 76.2 128.27 0)
       (effects (font (size 1.27 1.27)) hide)
     )
@@
   (symbol (lib_id "power:GND") (at 50.8 121.92 0) (unit 1)
     (in_bom yes) (on_board yes)
-    (property "Reference" "#PWR?" (id 0) (at 50.8 128.27 0)
+    (property "Reference" "#PWR0105" (id 0) (at 50.8 128.27 0)
       (effects (font (size 1.27 1.27)) hide)
     )
@@
   )
   (symbol_instances
+    (path "/b4420c8d-3935-4603-a990-13c1cb4fecdb"
+      (reference "#PWR0101") (unit 1) (value "GND") (footprint "")
+    )
+    (path "/24c2d2cf-16de-462d-8fd4-151ef01fc97c"
+      (reference "#PWR0102") (unit 1) (value "VCC") (footprint "")
+    )
+    (path "/bd363a98-b7ff-4a61-853f-37ae7b18e643"
+      (reference "#PWR0103") (unit 1) (value "GND") (footprint "")
+    )
+    (path "/062bb37c-0b34-45bf-a3bb-61501cc11844"
+      (reference "#PWR0104") (unit 1) (value "GND") (footprint "")
+    )
+    (path "/d1ca6120-06c9-4651-995d-ca0be7881930"
+      (reference "#PWR0105") (unit 1) (value "GND") (footprint "")
+    )
     (path "/00000000-0000-0000-0000-000062e1e0ee"
       (reference "#PWR0106") (unit 1) (value "VCC") (footprint "")
@@
       (reference "#PWR0115") (unit 1) (value "VCC") (footprint "")
     )
-    (path "/062bb37c-0b34-45bf-a3bb-61501cc11844"
-      (reference "#PWR?") (unit 1) (value "GND") (footprint "")
-    )
-    (path "/24c2d2cf-16de-462d-8fd4-151ef01fc97c"
-      (reference "#PWR?") (unit 1) (value "VCC") (footprint "")
-    )
-    (path "/b4420c8d-3935-4603-a990-13c1cb4fecdb"
-      (reference "#PWR?") (unit 1) (value "GND") (footprint "")
-    )
-    (path "/bd363a98-b7ff-4a61-853f-37ae7b18e643"
-      (reference "#PWR?") (unit 1) (value "GND") (footprint "")
-    )
-    (path "/d1ca6120-06c9-4651-995d-ca0be7881930"
-      (reference "#PWR?") (unit 1) (value "GND") (footprint "")
-    )
     (path "/9b6b6cbf-1b99-4cd5-865d-032611ca9f97"
       (reference "D0") (unit 1) (value "LED") (footprint "LED_SMD:LED_PLCC-2")
@@
       (reference "R2") (unit 1) (value "Rf") (footprint "Helios:RS_0805")
     )
-    (path "/9210b7d5-4a3c-42da-a207-c6563600611c"
-      (reference "R2") (unit 1) (value "RL") (footprint "Helios:RS_0805")
-    )
-    (path "/0c5a3185-120f-43f8-bc82-7edbf44849a1"
-      (reference "R3") (unit 1) (value "Rpd") (footprint "Helios:RS_0805")
-    )
     (path "/e25a04ec-21c5-43dd-9303-6ad094206daf"
       (reference "R3") (unit 1) (value "Rf") (footprint "Helios:RS_0805")
     )
+    (path "/9210b7d5-4a3c-42da-a207-c6563600611c"
+      (reference "R4") (unit 1) (value "RL") (footprint "Helios:RS_0805")
+    )
+    (path "/0c5a3185-120f-43f8-bc82-7edbf44849a1"
+      (reference "R5") (unit 1) (value "Rpd") (footprint "Helios:RS_0805")
+    )
     (path "/00000000-0000-0000-0000-000062e1e0e7"
