File: Electrónica/Helios/Helios_PCB/Helios_PCB_emitter/Helios_PCB_emitter.kicad_pcb (KiCad board)
At the start: 2 copper layers, 34 x 29.5 mm, 12 parts, among them J1 Conn_01x03_Male, Q0 AO3400A

Commit message: Last changes V1.3
Parts:
- removed D4: LED, LED_SMD:LED_miniPLCC_2315_Handsoldering
- added G***: LOGO, LOGO, B.Cu at (174.6, 90.6)
- added G***: LOGO, LOGO, B.Cu at (174.8, 107.7)
- R1: moved to F.Cu
- moved R1 20.9 mm to (177.9, 104.4)
- moved G*** 0.30 mm to (178.2, 100.0)
Connections:
- J1 pad 2: LED -> SIG
- Q0 pad 1: LED -> SIG
- R1 pad 1: Net-(D4-Pad1) -> SIG
Routing:
- net LED: track 21.3 -> 0.00 mm
- net SIG: track 0.00 -> 16.4 mm
- net Net-(D4-Pad1): track 2.00 -> 0.00 mm
Other:
- board text added: "12V"
- board text added: "AE RESET"
- board text added: "Colabora:"
- board text added: "EMT"
- board text added: "V S G"
- board text removed: "Helios Emitter"
