File: Electrónica/Helios/Helios_PCB/Helios_PCB_emitter/Helios_PCB_emitter.kicad_pcb (KiCad board)
At the start: 2 copper layers, 34 x 29.5 mm, 13 parts, among them J1 Conn_01x03_Male, Q0 AO3400A

Commit message: Helios Panel
Parts:
- removed Q0: AO3400A, Package_TO_SOT_SMD:SOT-23
- added JP: SolderJumper_2_Open, Jumper:SolderJumper-2_P1.3mm_Open_Pad1.0x1.5mm, B.Cu at (159.2, 101.3)
- added Q1: MMBT3904, Package_TO_SOT_SMD:SOT-23, B.Cu at (178.2, 100.0)
- J1: value Conn_01x03_Male -> Conn_02x03_Counter_Clockwise; footprint Connector_PinHeader_2.54mm:PinHeader_1x03_P2.54mm_Vertical -> Connector_PinHeader_2.54mm:PinHeader_2x03_P2.54mm_Vertical
- R0, R1: moved to B.Cu
- moved G*** 25.3 mm to (155.1, 89.8)
- moved G*** 19.1 mm to (155.9, 109.8)
- moved G*** 15.2 mm to (174.4, 109.4)
- moved R0 7.19 mm to (159.2, 98.7), turned to 0 degrees
- moved R1 6.95 mm to (171.7, 101.2), turned to 0 degrees
- moved J1 1.25 mm to (162.5, 101.2)
- turned D0 to -135 degrees
- turned D2 to 45 degrees
Connections:
- D0 pad 1: Net-(D0-Pad1) -> Net-(D0-K)
- D0 pad 2: Net-(D0-Pad2) -> Net-(D0-A)
- D1 pad 1: Net-(D0-Pad2) -> Net-(D0-K)
- D1 pad 2: Net-(D1-Pad2) -> Net-(D0-A)
- D2 pad 1: Net-(D1-Pad2) -> Net-(D0-K)
- D2 pad 2: Net-(D2-Pad2) -> Net-(D0-A)
- D3 pad 1: Net-(D2-Pad2) -> Net-(D0-K)
- D3 pad 2: Net-(D3-Pad2) -> Net-(D0-A)
- J1 pad 2: SIG -> VCC
- J1 pad 3: GND -> S0
- R0 pad 1: Net-(D3-Pad2) -> Net-(D0-A)
- R1 pad 1: SIG -> S0
- R1 pad 2: GND -> Net-(Q1-B)
Routing:
- net Net-(D0-K): track 0.00 -> 76.5 mm, vias 0 -> 2
- net Net-(D0-A): track 0.00 -> 62.0 mm, vias 0 -> 1
- net Net-(D1-Pad2): track 34.1 -> 0.00 mm
- net Net-(D0-Pad2): track 24.6 -> 0.00 mm
- net Net-(D2-Pad2): track 24.4 -> 0.00 mm
- net SIG: track 16.4 -> 0.00 mm
- net S0: track 0.00 -> 14.9 mm
- net Net-(D0-Pad1): track 9.39 -> 0.00 mm
- net Net-(D3-Pad2): track 7.38 -> 0.00 mm
- net Net-(Q1-B): track 0.00 -> 5.50 mm
- net VCC: track 11.2 -> 7.60 mm
Other:
- board text added: "Helios V2.1 2023"
- board text added: "V S1 G V S0 G"
- board text removed: "12V"
- board text removed: "AE RESET"
- board text removed: "EMT"
- board text removed: "G S V"
- board text removed: "Helios V1.3 2022"
- board text removed: "V S G"
