File: Electrónica/Helios/Helios_PCB/Helios_PCB_emitter/Helios_PCB_emitter.kicad_sch (KiCad schematic)
At the start: 9 parts, among them J1 Conn_01x03_Male, Q0 AO3400A

Commit message: Last changes V1.3
Parts:
- removed D4: LED, LED_SMD:LED_miniPLCC_2315_Handsoldering, symbol Device:LED
Connections:
- net LED is gone; now on net SIG: J1.2 (Pin_2), Q0.1 (G)
- net SIG: now reaches R1.1
Other:
- moved on the sheet: R1
Changed lines of the file:
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@@
     (stroke (width 0) (type default) (color 0 0 0 0))
   )
-  (wire (pts (xy 48.26 113.03) (xy 48.26 114.3))
+  (wire (pts (xy 48.26 109.22) (xy 48.26 114.3))
     (stroke (width 0) (type default) (color 0 0 0 0))
   )
@@
     (stroke (width 0) (type default) (color 0 0 0 0))
   )
-  (wire (pts (xy 48.26 93.98) (xy 48.26 96.52))
+  (wire (pts (xy 48.26 93.98) (xy 48.26 101.6))
     (stroke (width 0) (type default) (color 0 0 0 0))
   )
@@
     (stroke (width 0) (type default) (color 0 0 0 0))
   )
-  (wire (pts (xy 48.26 104.14) (xy 48.26 105.41))
-    (stroke (width 0) (type default) (color 0 0 0 0))
-  )
   (wire (pts (xy 114.3 91.44) (xy 109.22 91.44))
     (stroke (width 0) (type default) (color 0 0 0 0))
@@
     (stroke (width 0) (type default) (color 0 0 0 0))
   )
-  (global_label "LED" (shape input) (at 39.37 93.98 180) (fields_autoplaced)
+  (global_label "SIG" (shape input) (at 39.37 93.98 180) (fields_autoplaced)
     (effects (font (size 1.27 1.27)) (justify right))
-    (property "Intersheet References" "${INTERSHEET_REFS}" (id 0) (at 218.44 289.56 0)
-      (effects (font (size 1.27 1.27)) hide)
-    )
-  )
-  (global_label "LED" (shape input) (at 114.3 93.98 0) (fields_autoplaced)
+    (property "Intersheet References" "${INTERSHEET_REFS}" (id 0) (at 33.8726 93.9006 0)
+      (effects (font (size 1.27 1.27)) (justify right) hide)
+    )
+  )
+  (global_label "SIG" (shape input) (at 114.3 93.98 0) (fields_autoplaced)
     (effects (font (size 1.27 1.27)) (justify left))
-    (property "Intersheet References" "${INTERSHEET_REFS}" (id 0) (at -64.77 -101.6 0)
-      (effects (font (size 1.27 1.27)) hide)
-    )
-  )
-  (symbol (lib_id "Device:R") (at 48.26 109.22 0) (unit 1)
-    (in_bom yes) (on_board yes) (fields_autoplaced)
-    (property "Reference" "R1" (id 0) (at 50.038 109.6538 0)
+    (property "Intersheet References" "${INTERSHEET_REFS}" (id 0) (at 119.7974 93.9006 0)
+      (effects (font (size 1.27 1.27)) (justify left) hide)
+    )
+  )
+  (symbol (lib_id "Device:R") (at 48.26 105.41 0) (unit 1)
+    (in_bom yes) (on_board yes) (fields_autoplaced)
+    (property "Reference" "R1" (id 0) (at 50.038 105.8438 0)
       (effects (font (size 1.27 1.27)) (justify left))
     )
-    (property "Value" "Rpd" (id 1) (at 50.038 110.9222 0)
+    (property "Value" "Rpd" (id 1) (at 50.038 107.1122 0)
       (effects (font (size 1.27 1.27)) (justify left) hide)
     )
-    (property "Footprint" "Helios:RS_0805" (id 2) (at 46.482 109.22 90)
-      (effects (font (size 1.27 1.27)) hide)
-    )
-    (property "Datasheet" "~" (id 3) (at 48.26 109.22 0)
+    (property "Footprint" "Helios:RS_0805" (id 2) (at 46.482 105.41 90)
+      (effects (font (size 1.27 1.27)) hide)
+    )
+    (property "Datasheet" "~" (id 3) (at 48.26 105.41 0)
       (effects (font (size 1.27 1.27)) hide)
     )
@@
     (pin "1")
   )
-  (symbol (lib_id "Device:LED") (at 48.26 100.33 90) (unit 1)
-    (in_bom yes) (on_board yes) (fields_autoplaced)
-    (property "Reference" "D4" (id 0) (at 51.181 101.0828 90)
-      (effects (font (size 1.27 1.27)) (justify right))
-    )
-    (property "Value" "LED" (id 1) (at 51.181 103.6197 90)
-      (effects (font (size 1.27 1.27)) (justify right))
-    )
-    (property "Footprint" "LED_SMD:LED_miniPLCC_2315_Handsoldering" (id 2) (at 48.26 100.33 0)
-      (effects (font (size 1.27 1.27)) hide)
-    )
-    (property "Datasheet" "~" (id 3) (at 48.26 100.33 0)
-      (effects (font (size 1.27 1.27)) hide)
-    )
-    (pin "1")
-    (pin "2")
-  )
   (symbol (lib_id "Device:LED") (at 63.5 80.01 90) (unit 1)
     (in_bom yes) (on_board yes) (fields_autoplaced)
@@
       (reference "D3") (unit 1) (value "LED") (footprint "LED_SMD:LED_PLCC-2")
     )
-    (path "/deed5a59-f174-441d-8ba4-96bdb444ad80"
-      (reference "D4") (unit 1) (value "LED") (footprint "LED_SMD:LED_miniPLCC_2315_Handsoldering")
-    )
     (path "/ad961c12-86ce-46ad-9394-a7de12020501"

Commit message: Helios Panel
Parts:
- removed J1: Conn_01x03_Male, Connector_PinHeader_2.54mm:PinHeader_1x03_P2.54mm_Vertical, symbol Connector:Conn_01x03_Male
- removed Q0: AO3400A, Package_TO_SOT_SMD:SOT-23, symbol Transistor_FET:AO3400A
- added J1: Conn_02x03_Counter_Clockwise, Connector_PinHeader_2.54mm:PinHeader_2x03_P2.54mm_Vertical, symbol Connector_Generic:Conn_02x03_Counter_Clockwise
- added JP1: SolderJumper_2_Open, Jumper:SolderJumper-2_P1.3mm_Open_Pad1.0x1.5mm, symbol Jumper:SolderJumper_2_Open
- added Q1: MMBT3904, Package_TO_SOT_SMD:SOT-23, symbol Transistor_BJT:MMBT3904
Connections:
- net GND: now also J1.5 (Pin_5), J1.6 (Pin_6), Q1.2 (E); no longer R1.2
- net VCC: now also J1.1 (Pin_1), J1.2 (Pin_2), JP1.1 (A)
- net at D1.1 (K): now also D0.1 (K), D2.1 (K), D3.1 (K), Q1.3 (C); no longer D0.2 (A)
- net at D1.2 (A): now also D0.2 (A), D2.2 (A), D3.2 (A), R0.1; no longer D2.1 (K)
- net SIG renamed S0
- net S0: now also J1.3 (Pin_3), JP1.2 (B)
- new net: Q1.1 (B), R1.2
- new net S1: J1.4 (Pin_4)
Other:
- moved on the sheet: D0, D1, D2, D3, R0, R1
