File: Electrónica/Helios/Helios_PCB/Helios_PCB_section/Helios_PCB_section.kicad_sch (KiCad schematic)
At the start: 9 parts, among them J1 Conn_01x02_Socket, J2 Conn_01x02_Socket, J3 Conn_01x02_Socket, J4 Conn_01x04_Pin, J5 Conn_01x04_Pin, J6 Conn_01x04_Pin, U1 Sparkfun_Pro_Micro

Commit message: Added IMU PCB, female connection 3d model, assemblies. Error detected: invert connectors in PCB Male
Parts:
- added J7: Conn_01x02_Socket, Connector_PinHeader_2.54mm:PinHeader_1x02_P2.54mm_Vertical, symbol Connector:Conn_01x02_Socket
Connections:
- net +12V is gone; now on net +5V: J1.2 (Pin_2), U1.24 (RAW)
- net +5V: now also J7.1 (Pin_1); no longer U1.21 (VCC)
- net GND: now also J7.2 (Pin_2)
- no-connect marks 5 -> 6
Changed lines of the file:
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@@
   (no_connect (at 162.56 90.17))
   (no_connect (at 132.08 85.09))
+  (no_connect (at 162.56 92.71))
   (wire (pts (xy 162.56 95.25) (xy 166.37 95.25))
     (stroke (width 0) (type default))
@@
     (stroke (width 0) (type default))
   )
-  (wire (pts (xy 162.56 92.71) (xy 166.37 92.71))
-    (stroke (width 0) (type default))
-  )
   (wire (pts (xy 186.69 113.03) (xy 190.5 113.03))
     (stroke (width 0) (type default))
@@
     (stroke (width 0) (type default))
   )
+  (wire (pts (xy 227.33 85.09) (xy 231.14 85.09))
+    (stroke (width 0) (type default))
+  )
   (wire (pts (xy 128.27 105.41) (xy 132.08 105.41))
     (stroke (width 0) (type default))
@@
   )
   (wire (pts (xy 128.27 97.79) (xy 132.08 97.79))
+    (stroke (width 0) (type default))
+  )
+  (wire (pts (xy 227.33 87.63) (xy 231.14 87.63))
     (stroke (width 0) (type default))
   )
@@
         (path "/48a2e939-e701-47dd-b50e-977aeeb0d1a3"
           (reference "H1") (unit 1)
+        )
+      )
+    )
+  )
+  (symbol (lib_id "power:+5V") (at 227.33 85.09 90) (unit 1)
+    (in_bom yes) (on_board yes) (dnp no)
+    (property "Reference" "#PWR03" (at 231.14 85.09 0)
+      (effects (font (size 1.27 1.27)) hide)
+    )
+    (property "Value" "+5V" (at 223.52 85.09 90)
+      (effects (font (size 1.27 1.27)) (justify left))
+    )
+    (property "Footprint" "" (at 227.33 85.09 0)
+      (effects (font (size 1.27 1.27)) hide)
+    )
+    (property "Datasheet" "" (at 227.33 85.09 0)
+      (effects (font (size 1.27 1.27)) hide)
+    )
+    (pin "1")
+    (instances
+      (project "Helios_PCB_section"
+        (path "/48a2e939-e701-47dd-b50e-977aeeb0d1a3"
+          (reference "#PWR03") (unit 1)
+        )
+      )
+    )
+  )
+  (symbol (lib_id "Connector:Conn_01x02_Socket") (at 236.22 85.09 0) (unit 1)
+    (in_bom yes) (on_board yes) (dnp no) (fields_autoplaced)
+    (property "Reference" "J7" (at 237.49 85.725 0)
+      (effects (font (size 1.27 1.27)) (justify left))
+    )
+    (property "Value" "Conn_01x02_Socket" (at 237.49 88.265 0)
+      (effects (font (size 1.27 1.27)) (justify left))
+    )
+    (property "Footprint" "Connector_PinHeader_2.54mm:PinHeader_1x02_P2.54mm_Vertical" (at 236.22 85.09 0)
+      (effects (font (size 1.27 1.27)) hide)
+    )
+    (property "Datasheet" "~" (at 236.22 85.09 0)
+      (effects (font (size 1.27 1.27)) hide)
+    )
+    (pin "1")
+    (pin "2")
+    (instances
+      (project "Helios_PCB_section"
+        (path "/48a2e939-e701-47dd-b50e-977aeeb0d1a3"
+          (reference "J7") (unit 1)
         )
       )
@@
     )
   )
-  (symbol (lib_id "power:+12V") (at 186.69 80.01 90) (unit 1)
+  (symbol (lib_id "power:GND") (at 166.37 87.63 90) (unit 1)
+    (in_bom yes) (on_board yes) (dnp no)
+    (property "Reference" "#PWR02" (at 172.72 87.63 0)
+      (effects (font (size 1.27 1.27)) hide)
+    )
+    (property "Value" "GND" (at 170.18 87.63 90)
+      (effects (font (size 1.27 1.27)) (justify right))
+    )
+    (property "Footprint" "" (at 166.37 87.63 0)
+      (effects (font (size 1.27 1.27)) hide)
+    )
+    (property "Datasheet" "" (at 166.37 87.63 0)
+      (effects (font (size 1.27 1.27)) hide)
+    )
+    (pin "1")
+    (instances
+      (project "Helios_PCB_section"
+        (path "/48a2e939-e701-47dd-b50e-977aeeb0d1a3"
+          (reference "#PWR02") (unit 1)
+        )
+      )
+    )
+  )
+  (symbol (lib_id "power:GND") (at 186.69 77.47 270) (unit 1)
+    (in_bom yes) (on_board yes) (dnp no)
+    (property "Reference" "#PWR06" (at 180.34 77.47 0)
+      (effects (font (size 1.27 1.27)) hide)
+    )
+    (property "Value" "GND" (at 182.88 77.47 90)
+      (effects (font (size 1.27 1.27)) (justify right))
+    )
+    (property "Footprint" "" (at 186.69 77.47 0)
+      (effects (font (size 1.27 1.27)) hide)
+    )
+    (property "Datasheet" "" (at 186.69 77.47 0)
+      (effects (font (size 1.27 1.27)) hide)
+    )
+    (pin "1")
+    (instances
+      (project "Helios_PCB_section"
+        (path "/48a2e939-e701-47dd-b50e-977aeeb0d1a3"
+          (reference "#PWR06") (unit 1)
+        )
+      )
+    )
+  )
+  (symbol (lib_id "power:+5V") (at 186.69 80.01 90) (unit 1)
     (in_bom yes) (on_board yes) (dnp no)
     (property "Reference" "#PWR05" (at 190.5 80.01 0)
       (effects (font (size 1.27 1.27)) hide)
     )
-    (property "Value" "+12V" (at 182.88 80.01 90)
+    (property "Value" "+5V" (at 182.88 80.01 90)
       (effects (font (size 1.27 1.27)) (justify left))
     )
@@
         (path "/48a2e939-e701-47dd-b50e-977aeeb0d1a3"
           (reference "#PWR05") (unit 1)
-        )
-      )
-    )
-  )
-  (symbol (lib_id "power:GND") (at 166.37 87.63 90) (unit 1)
-    (in_bom yes) (on_board yes) (dnp no)
-    (property "Reference" "#PWR02" (at 172.72 87.63 0)
-      (effects (font (size 1.27 1.27)) hide)
-    )
-    (property "Value" "GND" (at 170.18 87.63 90)
-      (effects (font (size 1.27 1.27)) (justify right))
-    )
-    (property "Footprint" "" (at 166.37 87.63 0)
-      (effects (font (size 1.27 1.27)) hide)
-    )
-    (property "Datasheet" "" (at 166.37 87.63 0)
-      (effects (font (size 1.27 1.27)) hide)
-    )
-    (pin "1")
-    (instances
-      (project "Helios_PCB_section"
-        (path "/48a2e939-e701-47dd-b50e-977aeeb0d1a3"
-          (reference "#PWR02") (unit 1)
-        )
-      )
-    )
-  )
-  (symbol (lib_id "power:GND") (at 186.69 77.47 270) (unit 1)
-    (in_bom yes) (on_board yes) (dnp no)
-    (property "Reference" "#PWR06" (at 180.34 77.47 0)
-      (effects (font (size 1.27 1.27)) hide)
-    )
-    (property "Value" "GND" (at 182.88 77.47 90)
-      (effects (font (size 1.27 1.27)) (justify right))
-    )
-    (property "Footprint" "" (at 186.69 77.47 0)
-      (effects (font (size 1.27 1.27)) hide)
-    )
-    (property "Datasheet" "" (at 186.69 77.47 0)
-      (effects (font (size 1.27 1.27)) hide)
-    )
-    (pin "1")
-    (instances
-      (project "Helios_PCB_section"
-        (path "/48a2e939-e701-47dd-b50e-977aeeb0d1a3"
-          (reference "#PWR06") (unit 1)
         )
       )
@@
     )
   )
-  (symbol (lib_id "power:+5V") (at 166.37 92.71 270) (unit 1)
-    (in_bom yes) (on_board yes) (dnp no)
-    (property "Reference" "#PWR03" (at 162.56 92.71 0)
-      (effects (font (size 1.27 1.27)) hide)
-    )
-    (property "Value" "+5V" (at 170.18 92.71 90)
-      (effects (font (size 1.27 1.27)) (justify left))
-    )
-    (property "Footprint" "" (at 166.37 92.71 0)
-      (effects (font (size 1.27 1.27)) hide)
-    )
-    (property "Datasheet" "" (at 166.37 92.71 0)
-      (effects (font (size 1.27 1.27)) hide)
-    )
-    (pin "1")
-    (instances
-      (project "Helios_PCB_section"
-        (path "/48a2e939-e701-47dd-b50e-977aeeb0d1a3"
-          (reference "#PWR03") (unit 1)
-        )
-      )
-    )
-  )
   (symbol (lib_id "power:+5V") (at 227.33 77.47 90) (unit 1)
     (in_bom yes) (on_board yes) (dnp no)
@@
     )
   )
-  (symbol (lib_id "power:+12V") (at 166.37 85.09 270) (unit 1)
+  (symbol (lib_id "Connector:Conn_01x02_Socket") (at 195.58 77.47 0) (unit 1)
+    (in_bom yes) (on_board yes) (dnp no) (fields_autoplaced)
+    (property "Reference" "J1" (at 196.85 78.105 0)
+      (effects (font (size 1.27 1.27)) (justify left))
+    )
+    (property "Value" "Conn_01x02_Socket" (at 196.85 80.645 0)
+      (effects (font (size 1.27 1.27)) (justify left))
+    )
+    (property "Footprint" "XTConnectors:XT30U-M_1x02_P5.0mm_Vertical" (at 195.58 77.47 0)
+      (effects (font (size 1.27 1.27)) hide)
+    )
+    (property "Datasheet" "~" (at 195.58 77.47 0)
+      (effects (font (size 1.27 1.27)) hide)
+    )
+    (pin "1")
+    (pin "2")
+    (instances
+      (project "Helios_PCB_section"
+        (path "/48a2e939-e701-47dd-b50e-977aeeb0d1a3"
+          (reference "J1") (unit 1)
+        )
+      )
+    )
+  )
+  (symbol (lib_id "power:GND") (at 227.33 87.63 270) (unit 1)
+    (in_bom yes) (on_board yes) (dnp no)
+    (property "Reference" "#PWR09" (at 220.98 87.63 0)
+      (effects (font (size 1.27 1.27)) hide)
+    )
+    (property "Value" "GND" (at 223.52 87.63 90)
+      (effects (font (size 1.27 1.27)) (justify right))
+    )
+    (property "Footprint" "" (at 227.33 87.63 0)
+      (effects (font (size 1.27 1.27)) hide)
+    )
+    (property "Datasheet" "" (at 227.33 87.63 0)
+      (effects (font (size 1.27 1.27)) hide)
+    )
+    (pin "1")
+    (instances
+      (project "Helios_PCB_section"
+        (path "/48a2e939-e701-47dd-b50e-977aeeb0d1a3"
+          (reference "#PWR09") (unit 1)
+        )
+      )
+    )
+  )
+  (symbol (lib_id "power:+5V") (at 166.37 85.09 270) (unit 1)
     (in_bom yes) (on_board yes) (dnp no)
     (property "Reference" "#PWR01" (at 162.56 85.09 0)
       (effects (font (size 1.27 1.27)) hide)
     )
-    (property "Value" "+12V" (at 170.18 85.09 90)
+    (property "Value" "+5V" (at 170.18 85.09 90)
       (effects (font (size 1.27 1.27)) (justify left))
     )
@@
         )
       )
-    )
-  )
-  (symbol (lib_id "Connector:Conn_01x02_Socket") (at 195.58 77.47 0) (unit 1)
-    (in_bom yes) (on_board yes) (dnp no) (fields_autoplaced)
-    (property "Reference" "J1" (at 196.85 78.105 0)
-      (effects (font (size 1.27 1.27)) (justify left))
-    )
-    (property "Value" "Conn_01x02_Socket" (at 196.85 80.645 0)
-      (effects (font (size 1.27 1.27)) (justify left))
-    )
-    (property "Footprint" "XTConnectors:XT30U-M_1x02_P5.0mm_Vertical" (at 195.58 77.47 0)
-      (effects (font (size 1.27 1.27)) hide)
-    )
-    (property "Datasheet" "~" (at 195.58 77.47 0)
-      (effects (font (size 1.27 1.27)) hide)
-    )
-    (pin "1")
-    (pin "2")
-    (instances
-      (project "Helios_PCB_section"
-        (path "/48a2e939-e701-47dd-b50e-977aeeb0d1a3"
-          (reference "J1") (unit 1)
-        )
-      )
