File: Electrónica/Helios/Helios_PCB/Helios_PCB_receiver/Helios_PCB_receiver.kicad_pcb (KiCad board)
At the start: 2 copper layers, 34 x 29.5 mm, 16 parts, among them J0 Connector, U0 OPA2380, U1 OPA2380

Commit message: Helios Panel
Parts:
- removed J0: Connector, Connector_PinHeader_2.54mm:PinHeader_2x03_P2.54mm_Vertical
- added J1: Conn_02x02_Odd_Even, Connector_PinHeader_2.54mm:PinHeader_2x02_P2.54mm_Vertical, F.Cu at (166.4, 101.4)
- added J2: Conn_02x02_Odd_Even, Connector_PinHeader_2.54mm:PinHeader_2x02_P2.54mm_Vertical, F.Cu at (161.2, 101.4)
Routing:
- net O0: track 13.8 -> 18.8 mm
- net O3: track 18.8 -> 15.7 mm
- net O1: track 18.9 -> 21.1 mm
Other:
- board text added: "0 1"
- board text added: "1 0"
- board text added: "2 3"
- board text added: "3 2"
- board text added: "GND"
- board text added: "Helios V2.1 2023"
- board text removed: "0 3 G"
- board text removed: "2 1 V"
- board text removed: "G 3 0"
- board text removed: "Helios V1.3 2022"
- board text removed: "RCV"
- board text removed: "V 1 2"
