File: Electrónica/Helios/Helios_PCB/Helios_PCB_female/Helios_PCB_female.kicad_pcb (KiCad board)
At the start: 2 copper layers, 38 x 38 mm, 8 parts, among them J1 Conn_01x02_Socket, J2 Conn_01x02_Socket, J3 Conn_01x02_Socket, J4 Conn_01x02_Socket, J7 Conn_01x02_Socket

Commit message: Helios Panel
Parts:
- added G***: LOGO, LOGO, F.Cu at (98.1, 103.6)
- added G***: LOGO, LOGO, F.Cu at (111.6, 103.5)
- added G***: LOGO, LOGO, F.Cu at (104.8, 104.1)
- added G***: LOGO, LOGO, F.Cu at (104.9, 74.1)
- added G***: LOGO, LOGO, F.Cu at (116.9, 99.4)
- moved J7 2.62 mm to (103.3, 95.1), turned to 90 degrees
Connections:
- J1 pad 1: GND -> SCL
- J1 pad 2: +5V -> SDA
- J3 pad 1: SCL -> GND
- J3 pad 2: SDA -> +5V
- J4 pad 1: SDA -> SDA1
- J4 pad 2: SCL -> SCL1
- J7 pad 1: SDA1 -> SDA
- J7 pad 2: SCL1 -> SCL
Routing:
- net +5V: track 41.5 -> 107.5 mm
- net SCL: track 26.5 -> 15.8 mm
- net SDA: track 26.8 -> 16.3 mm
- net SDA1: track 11.2 -> 6.66 mm
- net SCL1: track 10.9 -> 9.08 mm
Other:
- board text added: "5V GND"
- board text added: "AE_RESET"
- board text added: "Colabora:"
- board text added: "Helios V2.1 2023"
- board text added: "JaimeBravoAlgaba Helios_SoftRobot"
- board text added: "SCL1 SDA1"
- board text added: "SDA SCL"
- board text removed: "+5V"
- board text removed: "GND"

Commit message: PCBs ready for manufacturing
Parts:
- moved H2 1.42 mm to (115.9, 79.1)
- moved H1 1.35 mm to (94.0, 100.9)
- renumbered MPU6050 to MPU1
Connections:
- J1 pad 1: SCL -> GND
- J1 pad 2: SDA -> +5V
- J3 pad 1: GND -> SCL
- J3 pad 2: +5V -> SDA
Routing:
- net +5V: track 107.5 -> 31.6 mm
- net SCL: track 15.8 -> 28.1 mm
- net SDA: track 16.3 -> 21.9 mm
Changed lines of the file:
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@@
   )
   (footprint "MountingHole:MountingHole_2.2mm_M2" (layer "F.Cu")
-    (at 93 100)
+    (at 94 100.9)
     (descr "Mounting Hole 2.2mm, no annular, M2")
     (tags "mounting hole 2.2mm no annular m2")
@@
       (stroke (width 0.1) (type solid)) (layer "F.Fab"))
     (pad "1" thru_hole rect (at 0 0 270) (size 3.8 3.8) (drill 2.7) (layers "*.Cu" "*.Mask")
-      (net 10 "SCL") (pinfunction "Pin_1") (pintype "passive"))
+      (net 5 "GND") (pinfunction "Pin_1") (pintype "passive"))
     (pad "2" thru_hole circle (at 5 0 270) (size 3.8 3.8) (drill 2.7) (layers "*.Cu" "*.Mask")
-      (net 9 "SDA") (pinfunction "Pin_2") (pintype "passive"))
+      (net 6 "+5V") (pinfunction "Pin_2") (pintype "passive"))
     (model "D:/Repositorios/kicad-lib-amass_connectors/Connector_AMASS.3dshapes/Amass_XT30UPB-M.wrl"
       (offset (xyz 2.5 0 0))
@@
   )
   (footprint "MountingHole:MountingHole_2.2mm_M2" (layer "F.Cu")
-    (at 117 80)
+    (at 115.9 79.1)
     (descr "Mounting Hole 2.2mm, no annular, M2")
     (tags "mounting hole 2.2mm no annular m2")
@@
       (stroke (width 0.1) (type solid)) (layer "F.Fab"))
     (pad "1" thru_hole rect (at 0 0 270) (size 3.8 3.8) (drill 2.7) (layers "*.Cu" "*.Mask")
-      (net 5 "GND") (pinfunction "Pin_1") (pintype "passive"))
+      (net 10 "SCL") (pinfunction "Pin_1") (pintype "passive"))
     (pad "2" thru_hole circle (at 5 0 270) (size 3.8 3.8) (drill 2.7) (layers "*.Cu" "*.Mask")
-      (net 6 "+5V") (pinfunction "Pin_2") (pintype "passive"))
+      (net 9 "SDA") (pinfunction "Pin_2") (pintype "passive"))
     (model "D:/Repositorios/kicad-lib-amass_connectors/Connector_AMASS.3dshapes/Amass_XT30UPB-M.wrl"
       (offset (xyz 2.5 0 0))
@@
     (property "Sheetname" "")
     (attr through_hole)
-    (fp_text reference "MPU6050" (at -1.225 9.695 unlocked) (layer "F.SilkS")
+    (fp_text reference "MPU1" (at -1.225 9.695 unlocked) (layer "F.SilkS")
         (effects (font (size 1 1) (thickness 0.1)))
     )
@@
   (gr_circle (center 105 90) (end 124 90)
     (stroke (width 0.15) (type default)) (fill none) (layer "Dwgs.User"))
+  (gr_line (start 105 90) (end 115.96 79.04)
+    (stroke (width 0.15) (type default)) (layer "Dwgs.User"))
   (gr_line (start 105 90) (end 130 115)
     (stroke (width 0.15) (type default)) (layer "Dwgs.User"))
+  (gr_circle (center 105 90) (end 89.5 90)
+    (stroke (width 0.15) (type default)) (fill none) (layer "Dwgs.User"))
   (gr_circle (center 105 90) (end 105 112)
     (stroke (width 0.15) (type default)) (fill none) (layer "Dwgs.User"))
@@
   (gr_circle (center 117.25 108.25) (end 116.25 108.25)
     (stroke (width 0.15) (type default)) (fill none) (layer "Dwgs.User"))
+  (gr_line (start 105 90) (end 94.04 100.96)
+    (stroke (width 0.15) (type default)) (layer "Dwgs.User"))
   (gr_circle (center 127 90) (end 127 88.5)
     (stroke (width 0.15) (type default)) (fill none) (layer "Dwgs.User"))
   (gr_circle (center 105 90) (end 130 90)
     (stroke (width 0.15) (type default)) (fill none) (layer "Dwgs.User"))
-  (gr_line (start 105 90) (end 117 80)
-    (stroke (width 0.15) (type default)) (layer "Dwgs.User"))
-  (gr_line (start 105 90) (end 93 100)
-    (stroke (width 0.15) (type default)) (layer "Dwgs.User"))
   (gr_line (start 105 90) (end 134 110)
     (stroke (width 0.15) (type default)) (layer "Dwgs.User"))
@@
   (gr_circle (center 105 90) (end 105 71)
     (stroke (width 0.1) (type default)) (fill none) (layer "Edge.Cuts"))
-  (gr_text " 5V    GND" (at 86.7156 94.3356 270) (layer "B.SilkS")
+  (gr_text " 5V    GND" (at 121.576 94.4048 270) (layer "B.SilkS")
     (effects (font (size 1 1) (thickness 0.15)) (justify left bottom mirror))
   )
@@
     (effects (font (size 1 1) (thickness 0.15)) (justify left bottom mirror))
   )
-  (gr_text "SDA    SCL" (at 121.7676 94.1324 270) (layer "B.SilkS")
+  (gr_text "SDA    SCL" (at 87.0284 94.1508 270) (layer "B.SilkS")
     (effects (font (size 1 1) (thickness 0.15)) (justify left bottom mirror))
   )
-  (gr_text " 5V    GND" (at 88.2396 94.0308 90) (layer "F.SilkS")
+  (gr_text " 5V    GND" (at 123.1 94.1 90) (layer "F.SilkS")
     (effects (font (size 1 1) (thickness 0.15)) (justify left bottom))
   )
@@
     (effects (font (size 0.5 0.5) (thickness 0.1) bold) (justify left bottom))
   )
-  (gr_text "SDA    SCL" (at 123.1392 94.0816 90) (layer "F.SilkS")
+  (gr_text "SDA    SCL" (at 88.4 94.1 90) (layer "F.SilkS")
     (effects (font (size 1 1) (thickness 0.15)) (justify left bottom))
   )
@@
     (effects (font (size 1 1) (thickness 0.15)) (justify mirror))
   )
-  (segment (start 95.38 89.795) (end 92.7 92.475) (width 2) (layer "F.Cu") (net 6))
-  (segment (start 95.38 79) (end 95.38 81.1) (width 2) (layer "F.Cu") (net 6))
-  (segment (start 97.15 77.23) (end 95.38 79) (width 2) (layer "F.Cu") (net 6))
-  (segment (start 95.38 81.1) (end 95.38 89.795) (width 2) (layer "F.Cu") (net 6))
-  (segment (start 111.23 87.09) (end 111.23 80.66) (width 2) (layer "F.Cu") (net 6))
-  (segment (start 98.38 77.24) (end 98.37 77.23) (width 1) (layer "F.Cu") (net 6))
-  (segment (start 111.28 80.61) (end 107.9 77.23) (width 2) (layer "F.Cu") (net 6))
-  (segment (start 111.23 80.66) (end 111.28 80.61) (width 2) (layer "F.Cu") (net 6))
-  (segment (start 98.37 77.23) (end 97.15 77.23) (width 2) (layer "F.Cu") (net 6))
-  (segment (start 95.3854 81.1054) (end 95.38 81.1) (width 1) (layer "F.Cu") (net 6))
-  (segment (start 106 89.8722) (end 108.4478 89.8722) (width 2) (layer "F.Cu") (net 6))
-  (segment (start 108.4478 89.8722) (end 111.23 87.09) (width 2) (layer "F.Cu") (net 6))
-  (segment (start 107.9 77.23) (end 98.37 77.23) (width 2) (layer "F.Cu") (net 6))
-  (segment (start 92.7 92.475) (end 91.5 92.475) (width 2) (layer "F.Cu") (net 6))
-  (segment (start 98.38 81.1054) (end 95.3854 81.1054) (width 1) (layer "F.Cu") (net 6))
-  (segment (start 98.38 81.1054) (end 98.38 77.24) (width 1) (layer "F.Cu") (net 6))
-  (segment (start 98.36 77.12) (end 97.1 77.12) (width 2) (layer "B.Cu") (net 6))
-  (segment (start 108.6078 89.8722) (end 111.21 87.27) (width 2) (layer "B.Cu") (net 6))
-  (segment (start 95.3654 81.1054) (end 95.33 81.07) (width 1) (layer "B.Cu") (net 6))
-  (segment (start 111.21 87.27) (end 111.21 80.59) (width 2) (layer "B.Cu") (net 6))
-  (segment (start 92.565 92.475) (end 91.5 92.475) (width 2) (layer "B.Cu") (net 6))
-  (segment (start 95.33 78.89) (end 95.33 81.07) (width 2) (layer "B.Cu") (net 6))
-  (segment (start 107.74 77.12) (end 98.36 77.12) (width 2) (layer "B.Cu") (net 6))
-  (segment (start 97.1 77.12) (end 95.33 78.89) (width 2) (layer "B.Cu") (net 6))
-  (segment (start 106 89.8722) (end 108.6078 89.8722) (width 2) (layer "B.Cu") (net 6))
-  (segment (start 98.38 81.1054) (end 98.38 77.14) (width 1) (layer "B.Cu") (net 6))
-  (segment (start 98.38 77.14) (end 98.36 77.12) (width 1) (layer "B.Cu") (net 6))
-  (segment (start 111.21 80.59) (end 107.74 77.12) (width 2) (layer "B.Cu") (net 6))
-  (segment (start 98.38 81.1054) (end 95.3654 81.1054) (width 1) (layer "B.Cu") (net 6))
-  (segment (start 95.33 89.71) (end 92.565 92.475) (width 2) (layer "B.Cu") (net 6))
-  (segment (start 95.33 81.07) (end 95.33 89.71) (width 2) (layer "B.Cu") (net 6))
+  (segment (start 106.0054 81.1054) (end 107.9 83) (width 1) (layer "F.Cu") (net 6))
+  (segment (start 107.9 87.9722) (end 106 89.8722) (width 1) (layer "F.Cu") (net 6))
+  (segment (start 98.38 81.1054) (end 106.0054 81.1054) (width 1) (layer "F.Cu") (net 6))
+  (segment (start 107.9 83) (end 107.9 87.9722) (width 1) (layer "F.Cu") (net 6))
+  (segment (start 106 89.8722) (end 108.6278 92.5) (width 2) (layer "B.Cu") (net 6))
+  (segment (start 108.6278 92.5) (end 118.5 92.5) (width 2) (layer "B.Cu") (net 6))
   (segment (start 105.364081 86.46) (end 98.6546 86.46) (width 1) (layer "F.Cu") (net 7))
   (segment (start 105.913 85.911081) (end 105.364081 86.46) (width 1) (layer "F.Cu") (net 7))
@@
   (segment (start 103.373 84.709) (end 102.3964 84.709) (width 1) (layer "B.Cu") (net 8))
   (segment (start 102.3964 84.709) (end 98.38 88.7254) (width 1) (layer "B.Cu") (net 8))
-  (segment (start 105.865 92.5) (end 118.5 92.5) (width 1) (layer "B.Cu") (net 9))
-  (segment (start 103.305 95.06) (end 105.865 92.5) (width 1) (layer "B.Cu") (net 9))
-  (segment (start 110.94 95.06) (end 118.5 87.5) (width 1) (layer "F.Cu") (net 10))
-  (segment (start 105.845 95.06) (end 110.94 95.06) (width 1) (layer "F.Cu") (net 10))
+  (segment (start 100.2 101.5) (end 97.5 101.5) (width 1) (layer "B.Cu") (net 9))
+  (segment (start 97.5 101.5) (end 91.5 95.5) (width 1) (layer "B.Cu") (net 9))
+  (segment (start 103.305 95.06) (end 103.305 98.395) (width 1) (layer "B.Cu") (net 9))
+  (segment (start 91.5 95.5) (end 91.5 92.475) (width 1) (layer "B.Cu") (net 9))
+  (segment (start 103.305 98.395) (end 100.2 101.5) (width 1) (layer "B.Cu") (net 9))
+  (segment (start 100.4 101.5) (end 97.5 101.5) (width 1) (layer "F.Cu") (net 10))
+  (segment (start 95 99) (end 95 90.975) (width 1) (layer "F.Cu") (net 10))
+  (segment (start 105.845 96.055) (end 100.4 101.5) (width 1) (layer "F.Cu") (net 10))
+  (segment (start 95 90.975) (end 91.5 87.475) (width 1) (layer "F.Cu") (net 10))
+  (segment (start 105.845 95.06) (end 105.845 96.055) (width 1) (layer "F.Cu") (net 10))
+  (segment (start 97.5 101.5) (end 95 99) (width 1) (layer "F.Cu") (net 10))
   (zone (net 5) (net_name "GND") (layers "F&B.Cu") (hatch edge 0.5)
     (connect_pads (clearance 0.5))
