File: Electrónica/Helios/Helios_PCB/Helios_PCB_female/Helios_PCB_female.kicad_pcb (KiCad board)
At the start: 2 copper layers, 38 x 38 mm, 13 parts, among them J1 Conn_01x02_Socket, J2 Conn_01x02_Socket, J3 Conn_01x02_Socket, J4 Conn_01x02_Socket, J7 Conn_01x02_Socket

Commit message: V2.2 - BNO_055 IMU
Parts:
- removed MPU1: ~, MPU6050:MPU6050_module
- added BNO_055: ~, BNO_055:BNO_055, F.Cu at (105.1, 89.9)
Routing:
- net +5V: track 31.6 -> 41.1 mm
- net SCL1: track 9.08 -> 14.2 mm
- net SDA1: track 6.66 -> 9.82 mm
Other:
- board text added: "BNO_055"
- board text added: "Helios V2.2 2023"
- board text removed: "Helios V2.1 2023"
