File: Electrónica/Helios/Helios_PCB/Helios_PCB_panel/Helios_PCB_panel.kicad_pcb (KiCad board)
At the start: 2 copper layers, 160 x 160 mm, 51 parts, among them M0_0 Conn_01x04_Pin, M0_1 Conn_01x04_Pin, M0_2 Conn_01x04_Pin, M0_3 Conn_01x04_Pin, M1_0 Conn_01x04_Pin, M1_1 Conn_01x04_Pin, M1_2 Conn_01x04_Pin, M1_3 Conn_01x04_Pin, M2_0 Conn_01x04_Pin, M2_1 Conn_01x04_Pin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

Commit message: PCBs ready for manufacturing
Parts:
- I2C1: value 12VDC -> I2C1
- renumbered ESP32 to MCU1
Connections:
- I2C1 pad 1: SDA -> SCL
- I2C1 pad 2: SCL -> SDA
Routing:
- net SDA: track 35.3 -> 27.8 mm
- net S0: track 220.0 -> 215.9 mm
- net SCL: track 25.4 -> 29.4 mm
- net D1: track 282.7 -> 285.5 mm
- net S3: track 271.7 -> 274.4 mm
- net Net-(DRV2_1-A2): track 58.9 -> 56.4 mm
- net S2: track 225.2 -> 223.1 mm
- net S1: track 274.8 -> 276.6 mm
- net Net-(DRV2_1-B1): track 64.0 -> 62.5 mm
- net Net-(DRV1_0-A1): track 38.7 -> 40.1 mm
- net +5V: track 514.9 -> 513.6 mm
- net Net-(DRV1_2-B1): track 31.3 -> 32.3 mm
- net Net-(DRV0_1-A1): track 61.7 -> 62.7 mm
- net Net-(DRV0_3-B2): track 63.0 -> 63.9 mm
- net Net-(DRV2_1-B2): track 64.4 -> 65.2 mm
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